Commit message: Added LiDAR and Camera

File: delivery_bot/description/face.xacro (robot description, xacro)
@@ -5,5 +5,5 @@
         <parent link="chassis"/>
         <child link="left_eye"/>
-        <origin xyz="1.03 0.17 0.22"  rpy="0.0 -${pi/2} 0.0"/>
+        <origin xyz="1.03 0.17 0.25"  rpy="0.0 -${pi/2} 0.0"/>
     </joint>
     <link name="left_eye">
@@ -14,4 +14,12 @@
             <material name="black"/>
         </visual>
+        <collision>
+            <geometry>
+                <cylinder radius="0.1" length="0.06"/>
+            </geometry>
+        </collision>
+        <xacro:inertial_cylinder mass="0.05" radius="0.1" length="0.06">
+            <origin xyz="0.0 0.0 0.0" rpy="0.0 0.0 0.0"/>
+        </xacro:inertial_cylinder>
     </link>
     <!-- RIGHT EYE LINK -->
@@ -19,5 +27,5 @@
         <parent link="chassis"/>
         <child link="right_eye"/>
-        <origin xyz="1.03 -0.17 0.22"  rpy="0.0 -${pi/2} 0.0"/>
+        <origin xyz="1.03 -0.17 0.25"  rpy="0.0 -${pi/2} 0.0"/>
     </joint>
     <link name="right_eye">
@@ -28,4 +36,12 @@
             <material name="black"/>
         </visual>
+        <collision>
+            <geometry>
+                <cylinder radius="0.1" length="0.06"/>
+            </geometry>
+        </collision>
+        <xacro:inertial_cylinder mass="0.05" radius="0.1" length="0.06">
+            <origin xyz="0.0 0.0 0.0" rpy="0.0 0.0 0.0"/>
+        </xacro:inertial_cylinder>
     </link>
     <!-- INNER LEFT EYE LINK -->
@@ -42,4 +58,12 @@
             <material name="glowing_blue"/>
         </visual>
+        <collision>
+            <geometry>
+                <cylinder radius="0.03" length="0.01"/>
+            </geometry>
+        </collision>
+        <xacro:inertial_cylinder mass="0.01" radius="0.03" length="0.01">
+            <origin xyz="0.0 0.0 0.0" rpy="0.0 0.0 0.0"/>
+        </xacro:inertial_cylinder>
     </link>
     <!-- INNER RIGHT EYE LINK -->
@@ -56,4 +80,12 @@
             <material name="glowing_blue"/>
         </visual>
+        <collision>
+            <geometry>
+                <cylinder radius="0.03" length="0.01"/>
+            </geometry>
+        </collision>
+        <xacro:inertial_cylinder mass="0.01" radius="0.03" length="0.01">
+            <origin xyz="0.0 0.0 0.0" rpy="0.0 0.0 0.0"/>
+        </xacro:inertial_cylinder>
     </link>
 </robot>

File: delivery_bot/description/robot.urdf.xacro (robot description, xacro)
@@ -2,5 +2,10 @@
 <robot xmlns:xacro="http://www.ros.org/wiki/xacro" name="delivery_bot">
     <xacro:include filename="colors.xacro"/>
+    <xacro:include filename="inertial_macros.xacro"/>
     <xacro:include filename="robot_core.xacro"/>
+    <xacro:include filename="wheels.xacro"/>
     <xacro:include filename="face.xacro"/>
+    <xacro:include filename="gazebo_control.xacro"/>
+    <xacro:include filename="lidar.xacro"/>
+    <xacro:include filename="camera.xacro"/>
 </robot>

File: delivery_bot/description/robot_core.xacro (robot description, xacro)
@@ -24,64 +24,13 @@
             <material name="carbon_black"/>
         </visual>
-    </link>
-    <!-- LEFT WHEEL LINK -->
-    <joint name="left_wheel_joint" type="continuous">
-        <parent link="base_link"/>
-        <child link="left_wheel"/>
-        <origin xyz="0.0 0.4 0.0" rpy="-${pi/2} 0.0 0.0"/>
-        <axis xyz="0.0 0.0 1.0"/>
-    </joint>
-    <link name="left_wheel">
-        <visual>
+        <collision>
+            <origin xyz="0.5 0.0 0.2" rpy="0.0 0.0 0.0"/>
             <geometry>
-                <cylinder radius="0.14" length="0.1"/>
+                <box size="1.0 0.7 0.4"/>
             </geometry>
-            <material name="dark_gray"/>
-        </visual>
-    </link>
-    <!-- RIGHT WHEEL LINK -->
-    <joint name="right_wheel_joint" type="continuous">
-        <parent link="base_link"/>
-        <child link="right_wheel"/>
-        <origin xyz="0.0 -0.4 0.0" rpy="${pi/2} 0.0 0.0"/>
-        <axis xyz="0.0 0.0 -1.0"/>
-    </joint>
-    <link name="right_wheel">
-        <visual>
-            <geometry>
-                <cylinder radius="0.14" length="0.1"/>
-            </geometry>
-            <material name="dark_gray"/>
-        </visual>
-    </link>
-    <!-- LEFT CASTER WHEEL LINK -->
-    <joint name="left_caster_wheel_joint" type="continuous">
-        <parent link="base_link"/>
-        <child link="left_caster_wheel"/>
-        <origin xyz="0.6 0.4 0.0" rpy="-${pi/2} 0.0 0.0"/>
-        <axis xyz="0.0 0. 1.0"/>
-    </joint>
-    <link name="left_caster_wheel">
-        <visual>
-            <geometry>
-                <cylinder radius="0.14" length="0.1"/>
-            </geometry>
-            <material name="dark_gray"/>
-        </visual>
-    </link>
-    <!-- RIGHT CASTER WHEEL LINK -->
-    <joint name="right_caster_wheel_joint" type="continuous">
-        <parent link="base_link"/>
-        <child link="right_caster_wheel"/>
-        <origin xyz="0.6 -0.4 0.0" rpy="${pi/2} 0.0 0.0"/>
-        <axis xyz="0.0 0.0 -1.0"/>
-    </joint>
-    <link name="right_caster_wheel">
-        <visual>
-            <geometry>
-                <cylinder radius="0.14" length="0.1"/>
-            </geometry>
-            <material name="dark_gray"/>
-        </visual>
+        </collision>
+        <xacro:inertial_box mass="2" x="1" y="0.7" z="0.4">
+            <origin xyz="0.5 0.0 0.2" rpy="0.0 0.0 0.0"/>
+        </xacro:inertial_box>
     </link>
     <!-- ITEM BASKET LINK -->
@@ -99,4 +48,13 @@
             <material name="deep_sci_fi_blue"/>
         </visual>
+        <collision>
+            <origin xyz="0.35 0.0 0.3"/>
+            <geometry>
+                <box size="0.7 0.7 0.6"/>
+            </geometry>
+        </collision>
+        <xacro:inertial_box mass="3" x="0.7" y="0.7" z="0.6">
+            <origin xyz="0.35 0.0 0.3"/>
+        </xacro:inertial_box>
     </link>
 </robot>
