Commit message: Added SLAM and Autonomous Navigation

File: delivery_bot/description/lidar.xacro (robot description, xacro)
@@ -2,7 +2,7 @@
 <robot xmlns:xacro="http://www.ros.org/wiki/xacro">
     <joint name="laser_joint" type="fixed">
-        <parent link="chassis"/>
+        <parent link="basket"/>
         <child link="laser_frame"/>
-        <origin xyz="0.5 0.0 -0.05"/>
+        <origin xyz="0.4 0.0 0.45"/>
     </joint>
     <link name="laser_frame">
@@ -36,5 +36,5 @@
                 </scan>
                 <range>
-                    <min>0.7</min>
+                    <min>0.6</min>
                     <max>15</max>
                 </range>

File: delivery_bot/description/robot_core.xacro (robot description, xacro)
@@ -42,14 +42,14 @@
     <link name="basket">
         <visual>
-            <origin xyz="0.35 0.0 0.3"/>
+            <origin xyz="0.4 0.0 0.2"/>
             <geometry>
-                <box size="0.7 0.7 0.6"/>
+                <box size="0.8 0.7 0.4"/>
             </geometry>
             <material name="deep_sci_fi_blue"/>
         </visual>
         <collision>
-            <origin xyz="0.35 0.0 0.3"/>
+            <origin xyz="0.35 0.0 0.2"/>
             <geometry>
-                <box size="0.7 0.7 0.6"/>
+                <box size="0.8 0.7 0.4"/>
             </geometry>
         </collision>
